File: hardware/led_panel/led_panel.kicad_pcb (KiCad board)
At the start: 2 copper layers, 99 x 89 mm, 21 parts, among them J1 Screw_Terminal_01x04, J2 Meanwell LPV-100-12, J3 Screw_Terminal_01x04, Q1 IRLZ24NPBF, Q2 IRLZ24NPBF, Q3 IRLZ24NPBF, Q4 IRLZ24NPBF, Q5 IRLZ24NPBF, Q6 IRLZ24NPBF, SW1 JOYIT_040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

Commit message: minor fix
Other:
- board text added: "JLCJLCJLCJLC"
- board text added: "Led panel ver .9 alpha"
Changed lines of the file:
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@@
   (general
     (thickness 1.6)
-    (drawings 45)
+    (drawings 47)
     (tracks 98)
     (zones 0)
@@
   (page A4)
   (layers
-    (0 F.Cu mixed)
+    (0 F.Cu mixed hide)
     (31 B.Cu mixed hide)
     (32 B.Adhes user hide)
@@
   )
   (setup
-    (last_trace_width 2.5)
+    (last_trace_width 0.25)
     (user_trace_width 0.4)
     (user_trace_width 0.6)
@@
       (outputformat 1)
       (mirror false)
-      (drillshape 1)
+      (drillshape 0)
       (scaleselection 1)
-      (outputdirectory ""))
+      (outputdirectory "gerber/"))
   )
   (net 0 "")
@@
       (solder_mask_margin 2) (clearance 3))
   )
+  (gr_text "Led panel \nver .9 alpha" (at 99.770001 88.975001) (layer F.SilkS)
+    (effects (font (size 1.5 1.5) (thickness 0.3)))
+  )
+  (gr_text JLCJLCJLCJLC (at 139.140001 78.815001) (layer F.SilkS)
+    (effects (font (size 1.5 1.5) (thickness 0.3)))
+  )
   (gr_text + (at 112.860001 48.405001) (layer F.SilkS)
