File: hardware/led_panel/led_panel.kicad_pcb (KiCad board)
At the start: 2 copper layers, 99 x 89 mm, 21 parts, among them J1 Screw_Terminal_01x04, J2 Meanwell LPV-100-12, J3 Screw_Terminal_01x04, Q1 IRLZ24NPBF, Q2 IRLZ24NPBF, Q3 IRLZ24NPBF, Q4 IRLZ24NPBF, Q5 IRLZ24NPBF, Q6 IRLZ24NPBF, SW1 JOYIT_040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

Commit message: git ignore for kicad
Parts:
- removed SW1: JOYIT_040, Connector_PinHeader_2.54mm:PinHeader_1x05_P2.54mm_Vertical
- removed U3: OLED, Connector_PinHeader_2.54mm:PinHeader_1x04_P2.54mm_Vertical
- J1, J3: footprint TerminalBlock_RND:TerminalBlock_RND_205-00047_1x04_P5.00mm_Horizontal -> TerminalBlock_Phoenix:TerminalBlock_Phoenix_MKDS-1,5-4_1x04_P5.00mm_Horizontal
- J2: footprint TerminalBlock:TerminalBlock_Altech_AK300-2_P5.00mm -> TerminalBlock_Phoenix:TerminalBlock_Phoenix_MKDS-1,5-2_1x02_P5.00mm_Horizontal
- moved C2 168.2 mm to (270.5, 30.1), turned to 0 degrees
- moved H4 159.9 mm to (240.2, 49.2)
- moved Q6 139.1 mm to (239.4, 42.6), turned to 0 degrees
- moved C1 136.3 mm to (250.0, 42.0), turned to 0 degrees
- moved Q3 133.6 mm to (259.9, 30.8), turned to 0 degrees
- moved H1 125.6 mm to (217.1, 76.1)
- moved Q1 121.2 mm to (259.9, 36.8), turned to 0 degrees
- moved J1 116.9 mm to (216.1, 33.1), turned to 0 degrees
- moved U2 116.6 mm to (227.9, 42.6), turned to 0 degrees
- moved J2 115.8 mm to (216.1, 45.0), turned to 0 degrees
- moved J3 112.1 mm to (238.2, 33.1), turned to 0 degrees
- moved R6 110.6 mm to (226.2, 46.7)
- moved Q4 103.3 mm to (227.4, 54.5), turned to 0 degrees
- moved Q5 100.3 mm to (215.8, 60.5), turned to 0 degrees
- moved H3 73.1 mm to (228.7, 61.1)
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Routing:
- net /3V3: track 68.3 -> 0.00 mm
- net Net-(J3-Pad4): track 56.6 -> 0.00 mm
- net Net-(J1-Pad2): track 47.1 -> 0.00 mm
- net /5V: track 34.1 -> 0.00 mm
- net /ROT+: track 33.3 -> 0.00 mm
- net /ROT-: track 33.3 -> 0.00 mm
- net /BUTTON: track 30.3 -> 0.00 mm
- net /SDA: track 29.5 -> 0.00 mm
- net /SCL: track 29.5 -> 0.00 mm
- net Net-(J1-Pad3): track 29.1 -> 0.00 mm
- net /BLUE: track 28.2 -> 0.00 mm
- net /GREEN: track 27.1 -> 0.00 mm
- net Earth: track 26.7 -> 0.00 mm
- net Net-(J3-Pad3): track 24.8 -> 0.00 mm
- net Net-(J3-Pad2): track 20.0 -> 0.00 mm
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- removed copper zone on F.Cu, net +12V
- removed copper zone on B.Cu, net Earth
Other:
- board outline removed
- net class Default: clearance 0.1 -> 0.2
- rule pad_to_mask_clearance: 0.051 -> 0
- rule trace_clearance: 0.1 -> 0.2
- rule via_min_drill: 0.2 -> 0.3
- rule via_min_size: 0.45 -> 0.4
- board text removed: "+"
- board text removed: "+12"
- board text removed: "3V3"
- board text removed: "B"
- board text removed: "CLK"
- board text removed: "DT"
- board text removed: "G"
- board text removed: "GND"
- board text removed: "IRLZ24NPBF"
- board text removed: "JLCJLCJLCJLC"
- board text removed: "JOYIT 040 ROTARY"
- board text removed: "Led panel ver .9 alpha"
- board text removed: "NODEMCUV1"
- board text removed: "OLED"
- board text removed: "R"
- board text removed: "SCL"
- board text removed: "SDA"
- board text removed: "SW"
- board text removed: "VCC"

Commit message: kicad tidy
Parts:
- added SW1: JOYIT_040, Connector_PinHeader_2.54mm:PinHeader_1x05_P2.54mm_Vertical, F.Cu at (136.5, 63.0)
- added U3: OLED, Connector_PinHeader_2.54mm:PinHeader_1x04_P2.54mm_Vertical, F.Cu at (136.0, 83.5)
- U1: value NodeMCU1.0(ESP-12E) -> NodeMCU_1.0_(ESP-12E)
- moved Q3 172.7 mm to (96.0, 85.1), turned to 90 degrees
- moved Q1 167.9 mm to (96.0, 73.2), turned to 90 degrees
- moved H4 161.4 mm to (81.0, 22.5)
- moved J3 157.5 mm to (81.0, 44.0), turned to 270 degrees
- moved C2 149.0 mm to (121.5, 34.0)
- moved Q6 144.6 mm to (96.0, 61.3), turned to 90 degrees
- moved H2 139.3 mm to (81.0, 96.5)
- moved J1 139.2 mm to (81.0, 66.5), turned to 270 degrees
- moved Q4 131.5 mm to (96.0, 49.4), turned to 90 degrees
- moved Q5 125.3 mm to (96.0, 97.0), turned to 90 degrees
- moved Q2 121.0 mm to (96.0, 37.5), turned to 90 degrees
- moved C1 120.3 mm to (130.0, 34.0), turned to 180 degrees
- moved R6 114.2 mm to (112.6, 35.0), turned to 180 degrees
- moved J2 106.3 mm to (111.5, 26.0), turned to 180 degrees
- moved H3 105.0 mm to (131.0, 22.5)
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Connections:
- net /5V renamed +5V
- net /BLUE renamed BLUE
- net /GREEN renamed GREEN
- net /RED renamed RED
- U1 pad 10: Earth -> Net-(U1-Pad10)
- U1 pad 11: /3V3 -> +3V3
- U1 pad 16: /3V3 -> Net-(U1-Pad16)
- U1 pad 17: Earth -> Net-(U1-Pad17)
- U1 pad 19: /BUTTON -> BUTTON
- U1 pad 24: Earth -> Net-(U1-Pad24)
- U1 pad 26: /ROT- -> ROT-
- U1 pad 27: /ROT+ -> ROT+
- U1 pad 28: /SDA -> SDA
- U1 pad 29: /SCL -> SCL
Routing:
- net BLUE: track 0.00 -> 48.3 mm
- net GREEN: track 0.00 -> 47.5 mm
- net +5V: track 0.00 -> 47.0 mm
- net RED: track 0.00 -> 46.1 mm
- net BUTTON: track 0.00 -> 40.6 mm
- net ROT-: track 0.00 -> 40.0 mm
- net ROT+: track 0.00 -> 39.4 mm
- net +3V3: track 0.00 -> 39.4 mm
- net SDA: track 0.00 -> 34.7 mm
- net SCL: track 0.00 -> 34.7 mm
- net Net-(J3-Pad2): track 0.00 -> 23.7 mm
- net Net-(J1-Pad4): track 0.00 -> 23.0 mm
- net Net-(R5-Pad2): track 0.00 -> 18.2 mm
- net Net-(J3-Pad3): track 0.00 -> 18.0 mm
- net Net-(J1-Pad3): track 0.00 -> 17.5 mm
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- added copper zone on F.Cu, net +12V
- added copper zone on B.Cu, net Earth
Other:
- board outline added: 67.5 x 86 mm
