File: hardware/led_panel/led_panel.sch (KiCad schematic (older format))
At the start: 21 parts, among them J1 Screw_Terminal_01x04, J2 Meanwell LPV-100-12, J3 Screw_Terminal_01x04, Q1 IRLZ24NPBF, Q2 IRLZ24NPBF, Q3 IRLZ24NPBF, Q4 IRLZ24NPBF, Q5 IRLZ24NPBF, Q6 IRLZ24NPBF, SW1 JOYIT_040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

Commit message: minor fix
Connections:
- net 3V3: no longer U1.25 (3.3V)
- no-connect marks 14 -> 15
Changed lines of the file:
@@
 Text Label 2300 6750 0    50   ~ 10
 GND
-Text Label 2300 6650 0    50   ~ 10
-3V3
 Text Label 2300 7550 0    50   ~ 10
 3V3
@@
 Wire Wire Line
 	5600 2700 5850 2700
+NoConn ~ 2300 6650
 $EndSCHEMATC

Commit message: git ignore for kicad
Parts:
- J1, J3: footprint TerminalBlock_Dinkle:TerminalBlock_Dinkle_DT-55-B01X-04_P10.00mm -> TerminalBlock_Phoenix:TerminalBlock_Phoenix_MKDS-1,5-4_1x04_P5.00mm_Horizontal
- J2: footprint TerminalBlock:TerminalBlock_Altech_AK300-2_P5.00mm -> TerminalBlock_Phoenix:TerminalBlock_Phoenix_MKDS-1,5-2_1x02_P5.00mm_Horizontal
Other:
- moved on the sheet: H1, H2, H3, H4
Changed lines of the file:
@@
 EESchema Schematic File Version 4
-EELAYER 26 0
+EELAYER 30 0
 EELAYER END
 $Descr A4 11693 8268
@@
 F 0 "J2" H 950 1000 50  0000 C CNN
 F 1 "Meanwell LPV-100-12" H 950 1350 50  0000 C CNN
-F 2 "TerminalBlock:TerminalBlock_Altech_AK300-2_P5.00mm" H 950 1200 50  0001 C CNN
+F 2 "TerminalBlock_Phoenix:TerminalBlock_Phoenix_MKDS-1,5-2_1x02_P5.00mm_Horizontal" H 950 1200 50  0001 C CNN
 F 3 "~" H 950 1200 50  0001 C CNN
 	1    950  1200
@@
 L Mechanical:MountingHole H1
 U 1 1 5F9B86AA
-P 10250 900
-F 0 "H1" H 10350 946 50  0000 L CNN
-F 1 "MountingHole" H 10350 855 50  0000 L CNN
-F 2 "MountingHole:MountingHole_4.3mm_M4_DIN965" H 10250 900 50  0001 C CNN
-F 3 "~" H 10250 900 50  0001 C CNN
-	1    10250 900
+P 10150 750
+F 0 "H1" H 10250 796 50  0000 L CNN
+F 1 "MountingHole" H 10250 705 50  0000 L CNN
+F 2 "MountingHole:MountingHole_4.3mm_M4_DIN965" H 10150 750 50  0001 C CNN
+F 3 "~" H 10150 750 50  0001 C CNN
+	1    10150 750
 	1    0    0    -1
 $EndComp
@@
 L Mechanical:MountingHole H2
 U 1 1 5F9B87AA
-P 10250 1100
-F 0 "H2" H 10350 1146 50  0000 L CNN
-F 1 "MountingHole" H 10350 1055 50  0000 L CNN
-F 2 "MountingHole:MountingHole_4.3mm_M4_DIN965" H 10250 1100 50  0001 C CNN
-F 3 "~" H 10250 1100 50  0001 C CNN
-	1    10250 1100
+P 10150 950
+F 0 "H2" H 10250 996 50  0000 L CNN
+F 1 "MountingHole" H 10250 905 50  0000 L CNN
+F 2 "MountingHole:MountingHole_4.3mm_M4_DIN965" H 10150 950 50  0001 C CNN
+F 3 "~" H 10150 950 50  0001 C CNN
+	1    10150 950
 	1    0    0    -1
 $EndComp
@@
 L Mechanical:MountingHole H3
 U 1 1 5F9B87EC
-P 10250 1300
-F 0 "H3" H 10350 1346 50  0000 L CNN
-F 1 "MountingHole" H 10350 1255 50  0000 L CNN
-F 2 "MountingHole:MountingHole_4.3mm_M4_DIN965" H 10250 1300 50  0001 C CNN
-F 3 "~" H 10250 1300 50  0001 C CNN
-	1    10250 1300
+P 10150 1150
+F 0 "H3" H 10250 1196 50  0000 L CNN
+F 1 "MountingHole" H 10250 1105 50  0000 L CNN
+F 2 "MountingHole:MountingHole_4.3mm_M4_DIN965" H 10150 1150 50  0001 C CNN
+F 3 "~" H 10150 1150 50  0001 C CNN
+	1    10150 1150
 	1    0    0    -1
 $EndComp
@@
 L Mechanical:MountingHole H4
 U 1 1 5F9B8838
-P 10250 1500
-F 0 "H4" H 10350 1546 50  0000 L CNN
-F 1 "MountingHole" H 10350 1455 50  0000 L CNN
-F 2 "MountingHole:MountingHole_4.3mm_M4_DIN965" H 10250 1500 50  0001 C CNN
-F 3 "~" H 10250 1500 50  0001 C CNN
-	1    10250 1500
+P 10150 1350
+F 0 "H4" H 10250 1396 50  0000 L CNN
+F 1 "MountingHole" H 10250 1305 50  0000 L CNN
+F 2 "MountingHole:MountingHole_4.3mm_M4_DIN965" H 10150 1350 50  0001 C CNN
+F 3 "~" H 10150 1350 50  0001 C CNN
+	1    10150 1350
 	1    0    0    -1
 $EndComp
@@
 F 0 "J1" V 2266 2162 50  0000 R CNN
 F 1 "Screw_Terminal_01x04" V 2175 2162 50  0000 R CNN
-F 2 "TerminalBlock_Dinkle:TerminalBlock_Dinkle_DT-55-B01X-04_P10.00mm" H 2300 2450 50  0001 C CNN
+F 2 "TerminalBlock_Phoenix:TerminalBlock_Phoenix_MKDS-1,5-4_1x04_P5.00mm_Horizontal" H 2300 2450 50  0001 C CNN
 F 3 "~" H 2300 2450 50  0001 C CNN
 	1    2300 2450
@@
 F 0 "J3" V 5916 2212 50  0000 R CNN
 F 1 "Screw_Terminal_01x04" V 5825 2212 50  0000 R CNN
-F 2 "TerminalBlock_Dinkle:TerminalBlock_Dinkle_DT-55-B01X-04_P10.00mm" H 5950 2500 50  0001 C CNN
+F 2 "TerminalBlock_Phoenix:TerminalBlock_Phoenix_MKDS-1,5-4_1x04_P5.00mm_Horizontal" H 5950 2500 50  0001 C CNN
 F 3 "~" H 5950 2500 50  0001 C CNN
 	1    5950 2500

Commit message: kicad tidy
Parts:
- removed U1: NodeMCU1.0(ESP-12E), ESP8266:ESP12F-Devkit-V3, symbol ESP8266:NodeMCU1.0(ESP-12E)
- added U1: NodeMCU_1.0_(ESP-12E), ESP8266:ESP12F-Devkit-V3, symbol ESP8266:NodeMCU_1.0_(ESP-12E)
- SW1: symbol oled:JOYIT_040 -> modules:Joyit_040_ENCODER
- U3: symbol oled:OLED -> modules:OLED
Connections:
- net BLUE: now also U1.21 (D7(GPIO13))
- net BUTTON: now also U1.19 (RX(DPIO3))
- net Earth: now also U1.14 (GND)
- net GREEN: now also U1.23 (D5(GPIO14))
- net RED: now also U1.22 (D6(GPIO12))
- net ROT+: now also U1.27 (D3(GPIO0))
- net ROT-: now also U1.26 (D4(GPIO2))
- net SCL: now also U1.29 (D1(GPIO5))
- net SDA: now also U1.28 (D2(GPIO4))
- net 3V3 renamed +3V3
- net +3V3: now also U1.11 (3.3V)
- net 5V renamed +5V
- net +5V: now also U1.15 (VIN)
- no-connect marks 15 -> 19
Other:
- note added: "LED strip connection and MOSFET drivers\n"
- note added: "M4"
- note added: "OLED display 168 x 64"
- note added: "ROT encoder"
- moved on the sheet: H1, H2, H3, H4, J1, Q1, Q3, Q5, SW1
